File: hardware/nrf24l01-stick.kicad_sch (KiCad schematic)
At the start: 25 parts, among them J1 USB_B_Micro, J2 SWD, SW1 SW_Push, U1 STM32L082KBUx, U2 NRF24L01_Breakout, U3 LP2985-3.3

Commit message: Designed the rest of the PCB.
Parts:
- removed C4: 0.01uF, Capacitor_SMD:C_0805_2012Metric, symbol Device:C
- removed C9: 10uF, Capacitor_SMD:C_0805_2012Metric, symbol Device:C
- removed R6: 1.5K, Resistor_SMD:R_0603_1608Metric, symbol Device:R
- removed U3: LP2985-3.3, Package_TO_SOT_SMD:SOT-23-5, symbol Regulator_Linear:LP2985-3.3
- added U3: MIC5504-3.3YM5, Package_TO_SOT_SMD:SOT-23-5, symbol Regulator_Linear:MIC5504-3.3YM5
- D1, D2: footprint LED_SMD:LED_0805_2012Metric -> LED_SMD:LED_0603_1608Metric
- R4, R5: value 20 -> 22
Connections:
- net +3V3: now also U3.5 (VOUT)
- net +5V: now also U3.1 (VIN), U3.3 (EN)
- net GND: now also U3.2 (GND)
- net ~IRQ: now also U1.9 (PA3); no longer U1.18 (PA8)
Other:
- note removed: "LP2992? Pin-compatible."
- moved on the sheet: C1, C2
